File: Schematic/Schematic.sch (KiCad schematic (older format))
At the start: 10 parts

Commit message: Added: shorter wait time for debug purposes, also close connection after every send.
Parts:
- removed BT?: Battery, symbol Device:Battery
- removed C? (x2): CAP, symbol pspice:CAP
- removed R?: R, symbol Device:R
- removed U?: SIM800C, RF_GSM:SIMCom_SIM800C, symbol RF_GSM:SIM800C
- added BT?: Battery_Cell, symbol Device:Battery_Cell
- added C?: CP_Small, symbol Device:CP_Small
- added U?: SIM800L, symbol Zander-Components:SIM800L
- A?: symbol MCU_Module:Arduino_Nano_Every -> Schematic-rescue:Arduino_Nano_Every-MCU_Module
Connections:
- wire segments 66 -> 62
Other:
- moved on the sheet: A?, J?, U?
